File: _autosave-PCBv1.kicad_pcb (KiCad board)
At the start: 2 copper layers, 157 parts, among them J1 AVR-ISP-6, SW1 `~, SW10 #8, SW11 #9, SW12 #0, SW13 -_, SW14 =+, SW15 BSPC, SW16 PAUSE, SW17 TAB, SW18 Q, SW19 W, SW2 SW_Push_Reset, SW20 E, SW21 R, SW22 T, SW23 Y, SW24 U, SW25 I, SW26 O, SW27 P, SW28 [{, SW29 ]}, SW3 #1, SW30 \|, SW31 NEXT, SW32 CPSLCK, SW33 A, SW34 S, SW35 D, SW36 F, SW37 G, SW38 H, SW39 J, SW4 #2, SW40 K, SW41 L, SW42 ;:, SW43 '", SW44 ENTR, SW45 PRVS, SW46 SHFT, SW47 Z, SW48 X, SW49 C, SW5 #3, SW50 V, SW51 B, SW52 N, SW53 M, SW54 ,<, SW55 .>, SW56 /?, SW57 SHFT, SW58 UP, SW59 DEL, SW6 #4, SW60 CTRL, SW61 WIN, SW62 ALT, SW63 SPC, SW64 ALT, SW65 FN, SW66 CTRL, SW67 LEFT, SW68 DOWN, SW69 RIGHT, SW7 #5, SW8 #6, SW9 #7, U1 ATmega32U4-A, Y1 16MHz

Commit message: pcb start
Parts:
- moved D16 250.0 mm to (281.0, 28.5), turned to 90 degrees
- moved D45 249.4 mm to (281.0, 66.6), turned to 90 degrees
- moved D59 249.4 mm to (281.0, 85.7), turned to 90 degrees
- moved D69 245.6 mm to (281.0, 104.8), turned to 90 degrees
- moved D58 230.6 mm to (261.9, 85.7), turned to 90 degrees
- moved D30 228.1 mm to (257.2, 47.6), turned to 90 degrees
- moved D68 226.5 mm to (261.9, 104.7), turned to 90 degrees
- moved D44 220.6 mm to (250.0, 66.6), turned to 90 degrees
- moved D13 209.0 mm to (204.8, 28.5), turned to 90 degrees
- moved D67 207.4 mm to (242.9, 104.7), turned to 90 degrees
- moved D31 207.0 mm to (135.1, -21.6), turned to 90 degrees
- moved D57 205.6 mm to (235.7, 85.7), turned to 90 degrees
- moved D12 195.0 mm to (185.7, 28.5), turned to 90 degrees
- moved D43 192.5 mm to (219.1, 66.6), turned to 90 degrees
- moved D29 191.1 mm to (135.2, -11.2), turned to 90 degrees
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