File: PCBv1.kicad_sch (KiCad schematic)
At the start: 14 parts, among them SW1 SW_Push, U1 ATmega32U4-A, Y1 16MHz

Commit message: asjkdhnasjkd
Parts:
- removed R2, R3: 22, symbol Device:R_Small
- removed R4: 10k, symbol Device:R_Small
- removed SW1: SW_Push, symbol Switch:SW_Push
- added D1: PRTR5V0U2X, Package_TO_SOT_SMD:SOT-143, symbol Power_Protection:PRTR5V0U2X
- added F1: 500m, symbol Device:Polyfuse_Small
- added J1: AVR-ISP-6, symbol Connector:AVR-ISP-6
- added R5: 10k, symbol Device:R_Small
- added R6, R7: 22, symbol Device:R_Small
- added R8, R9: 5.1k, symbol Device:R_Small
- added SW2: SW_Push_Reset, symbol Local:SW_SKQG
- added USB1: HRO-TYPE-C-31-M-12, symbol Type-C:HRO-TYPE-C-31-M-12
Connections:
- net +5V: now also F1.1, J1.2 (VCC), R5.1
- net D+: now also U1.4 (D+), R7.2
- net D-: now also U1.3 (D-), R6.2
- net GND: now also D1.1 (GND), J1.6 (GND), R8.1, R9.1, SW2. (2), USB1.1 (GND), USB1.12 (GND), USB1.13 (SHIELD)
- net RESET: now reaches U1.13 (~{RESET})
- net RESET: now also J1.5 (~{RST}), R5.2, SW2. (2)
- net MOSI: now reaches U1.10 (PB2)
- net MOSI: now also J1.4 (MOSI)
- net MISO: now reaches U1.11 (PB3)
- net MISO: now also J1.1 (MISO)
- net SCK: now reaches U1.9 (PB1)
- net SCK: now also J1.3 (SCK)
- new net: R8.2, USB1.10 (CC2)
- new net: R9.2, USB1.4 (CC1)
- new net: D1.3 (I/O2), R6.1, USB1.5 (DN2), USB1.7 (DN1)
- new net VCC: D1.2 (I/O1), D1.4 (VCC), F1.2, R7.1, USB1.11 (VBUS), USB1.2 (VBUS), USB1.6 (DP1), USB1.8 (DP2)
- no-connect marks 0 -> 4
Other:
- moved on the sheet: C1, C2, C3, C4, C5, C6, C7, R1, U1, Y1

Commit message: styuif
Other:
- added sheet matrix (matrix.kicad_sch)
Changed lines of the file:
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@@
+		)
+	)
+	(sheet
+		(at 163.83 108.585)
+		(size 46.355 23.495)
+		(exclude_from_sim no)
+		(in_bom yes)
+		(on_board yes)
+		(dnp no)
+		(fields_autoplaced yes)
+		(stroke
+			(width 0.1524)
+			(type solid)
+		)
+		(fill
+			(color 0 0 0 0.0000)
+		)
+		(property "Sheetname" "matrix"
+			(at 163.83 107.8734 0)
+			(effects
+				(font
+					(size 1.27 1.27)
+				)
+				(justify left bottom)
+			)
+		)
+		(property "Sheetfile" "matrix.kicad_sch"
+			(at 163.83 132.6646 0)
+			(effects
+				(font
+					(size 1.27 1.27)
+				)
+				(justify left top)
+			)
+		)
+		(instances
+			(project "PCBv1"
+				(path "/8d9d261d-9d52-405a-a0e1-e850188e3e4c"
+					(page "2")
+				)
+			)
 		)
 	)

Commit message: some progress
Connections:
- net row0: now reaches U1.1 (PE6)
- net col8: now reaches U1.19 (PD1)
- net col9: now reaches U1.20 (PD2)
- net col10: now reaches U1.21 (PD3)
- net col11: now reaches U1.22 (PD5)
- net col12: now reaches U1.25 (PD4)
- net col13: now reaches U1.26 (PD6)
- net col14: now reaches U1.27 (PD7)
- net col0: now reaches U1.28 (PB4)
- net col1: now reaches U1.29 (PB5)
- net col2: now reaches U1.30 (PB6)
- net col3: now reaches U1.31 (PC6)
- net col4: now reaches U1.32 (PC7)
- net col6: now reaches U1.36 (PF7)
- net col5: now reaches U1.37 (PF6)
- net row1: now reaches U1.38 (PF5)
- net row4: now reaches U1.39 (PF4)
- net row3: now reaches U1.40 (PF1)
- net row2: now reaches U1.41 (PF0)
- net col7: now reaches U1.8 (PB0)
- no-connect marks 4 -> 7

Commit message: pcb start
Parts:
- added C8: 0.1uF, Capacitor_SMD:C_0805_2012Metric_Pad1.18x1.45mm_HandSolder, symbol Device:C_Small
- C1, C2, C3, C4, C5, C6, C7: footprint (none) -> Capacitor_SMD:C_0805_2012Metric_Pad1.18x1.45mm_HandSolder
- F1: footprint (none) -> Fuse:Fuse_1206_3216Metric_Pad1.42x1.75mm_HandSolder
- J1: footprint (none) -> random-keyboard-parts:Reset_Pretty-Mask
- R1, R5, R6, R7, R8, R9: footprint (none) -> Resistor_SMD:R_0805_2012Metric_Pad1.20x1.40mm_HandSolder
- SW2: footprint (none) -> Button_Switch_SMD:SW_SPST_SKQG_WithStem
- USB1: footprint (none) -> Type-C:HRO-TYPE-C-31-M-12-HandSoldering
- Y1: footprint (none) -> Crystal:Crystal_SMD_3225-4Pin_3.2x2.5mm_HandSoldering
Connections:
- net +5V: now also C8.1
- net GND: now also C8.2
Changed lines of the file:
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@@
 	)
 	(junction
-		(at 34.29 86.36)
-		(diameter 0)
-		(color 0 0 0 0)
-	)
-	(junction
 		(at 72.39 166.37)
 		(diameter 0)
@@
 	)
 	(junction
-		(at 34.29 91.44)
-		(diameter 0)
-		(color 0 0 0 0)
-	)
-	(junction
 		(at 48.26 194.31)
 		(diameter 0)
@@
 	)
 	(junction
+		(at 21.59 86.36)
+		(diameter 0)
+		(color 0 0 0 0)
+	)
+	(junction
 		(at 55.88 194.31)
 		(diameter 0)
@@
 	)
 	(junction
+		(at 21.59 91.44)
+		(diameter 0)
+		(color 0 0 0 0)
+	)
+	(junction
 		(at 66.04 118.11)
 		(diameter 0)
@@
 	(wire
 		(pts
-			(xy 34.29 83.82) (xy 34.29 86.36)
+			(xy 30.48 83.82) (xy 30.48 86.36)
 		)
 		(stroke
@@
 	(wire
 		(pts
-			(xy 76.2 181.61) (xy 76.2 189.23)
+			(xy 13.97 86.36) (xy 21.59 86.36)
 		)
 		(stroke
@@
 	(wire
 		(pts
-			(xy 34.29 86.36) (xy 38.1 86.36)
+			(xy 76.2 181.61) (xy 76.2 189.23)
 		)
 		(stroke
@@
 	(wire
 		(pts
-			(xy 34.29 91.44) (xy 34.29 93.98)
+			(xy 30.48 91.44) (xy 30.48 93.98)
 		)
 		(stroke
@@
 	(wire
 		(pts
-			(xy 30.48 86.36) (xy 34.29 86.36)
+			(xy 30.48 86.36) (xy 38.1 86.36)
 		)
 		(stroke
@@
 	(wire
 		(pts
+			(xy 13.97 91.44) (xy 21.59 91.44)
+		)
+		(stroke
+			(width 0)
+			(type default)
+		)
+	)
+	(wire
+		(pts
 			(xy 53.34 189.23) (xy 53.34 181.61)
 		)
@@
 	(wire
 		(pts
+			(xy 30.48 91.44) (xy 38.1 91.44)
+		)
+		(stroke
+			(width 0)
+			(type default)
+		)
+	)
+	(wire
+		(pts
 			(xy 57.15 179.07) (xy 83.82 179.07)
 		)
@@
 	(wire
 		(pts
-			(xy 34.29 91.44) (xy 38.1 91.44)
-		)
-		(stroke
-			(width 0)
-			(type default)
-		)
-	)
-	(wire
-		(pts
 			(xy 66.04 171.45) (xy 66.04 186.69)
 		)
@@
 	(wire
 		(pts
-			(xy 30.48 91.44) (xy 34.29 91.44)
-		)
-		(stroke
-			(width 0)
-			(type default)
-		)
-	)
-	(wire
-		(pts
 			(xy 26.67 38.1) (xy 26.67 45.72)
 		)
@@
 			)
 		)
-		(property "Footprint" ""
+		(property "Footprint" "Capacitor_SMD:C_0805_2012Metric_Pad1.18x1.45mm_HandSolder"
 			(at 30.48 88.9 0)
 			(effects
@@
 			)
 		)
-		(property "Footprint" ""
+		(property "Footprint" "Resistor_SMD:R_0805_2012Metric_Pad1.20x1.40mm_HandSolder"
 			(at 95.25 87.63 0)
 			(effects
@@
 			)
 		)
-		(property "Footprint" ""
+		(property "Footprint" "Resistor_SMD:R_0805_2012Metric_Pad1.20x1.40mm_HandSolder"
 			(at 88.9 181.61 0)
 			(effects
@@
 			)
 		)
-		(property "Footprint" ""
+		(property "Footprint" "Type-C:HRO-TYPE-C-31-M-12-HandSoldering"
 			(at 44.45 177.8 0)
 			(effects
@@
 			)
 		)
-		(property "Footprint" ""
+		(property "Footprint" "Resistor_SMD:R_0805_2012Metric_Pad1.20x1.40mm_HandSolder"
 			(at 39.37 143.51 0)
 			(effects
@@
 			)
 		)
-		(property "Footprint" ""
+		(property "Footprint" "Resistor_SMD:R_0805_2012Metric_Pad1.20x1.40mm_HandSolder"
 			(at 88.9 179.07 0)
 			(effects
@@
 			)
 		)
-		(property "Footprint" ""
+		(property "Footprint" "Crystal:Crystal_SMD_3225-4Pin_3.2x2.5mm_HandSoldering"
 			(at 41.91 41.91 0)
 			(effects
@@
 			)
 		)
-		(property "Footprint" ""
+		(property "Footprint" "Capacitor_SMD:C_0805_2012Metric_Pad1.18x1.45mm_HandSolder"
 			(at 38.1 88.9 0)
 			(effects
@@
 			)
 		)
-		(property "Footprint" ""
+		(property "Footprint" "Capacitor_SMD:C_0805_2012Metric_Pad1.18x1.45mm_HandSolder"
 			(at 21.59 88.9 0)
 			(effects
@@
 			)
 		)
-		(property "Footprint" ""
+		(property "Footprint" "Capacitor_SMD:C_0805_2012Metric_Pad1.18x1.45mm_HandSolder"
 			(at 29.21 38.1 0)
 			(effects
@@
 			)
 		)
-		(property "Footprint" ""
+		(property "Footprint" "Button_Switch_SMD:SW_SPST_SKQG_WithStem"
 			(at 26.67 151.13 0)
 			(effects
@@
 			)
 		)
-		(property "Footprint" ""
+		(property "Footprint" "Capacitor_SMD:C_0805_2012Metric_Pad1.18x1.45mm_HandSolder"
 			(at 46.99 88.9 0)
 			(effects
@@
 			)
 		)
-		(property "Footprint" ""
+		(property "Footprint" "Resistor_SMD:R_0805_2012Metric_Pad1.20x1.40mm_HandSolder"
 			(at 66.04 189.23 0)
 			(effects
@@
 			)
 		)
-		(property "Footprint" ""
+		(property "Footprint" "Capacitor_SMD:C_0805_2012Metric_Pad1.18x1.45mm_HandSolder"
 			(at 41.91 69.85 0)
 			(effects
@@
 	(symbol
 		(lib_id "power:GND")
-		(at 34.29 93.98 0)
+		(at 30.48 93.98 0)
 		(unit 1)
 		(exclude_from_sim no)
@@
 		(fields_autoplaced yes)
 		(property "Reference" "#PWR06"
-			(at 34.29 100.33 0)
+			(at 30.48 100.33 0)
 			(effects
 				(font
@@
 		)
 		(property "Value" "GND"
-			(at 34.29 99.06 0)
+			(at 30.48 99.06 0)
 			(effects
 				(font
@@
 		)
 		(property "Footprint" ""
-			(at 34.29 93.98 0)
+			(at 30.48 93.98 0)
 			(effects
 				(font
@@
 		)
 		(property "Datasheet" ""
-			(at 34.29 93.98 0)
+			(at 30.48 93.98 0)
 			(effects
 				(font
@@
 		)
 		(property "Description" "Power symbol creates a global label with name \"GND\" , ground"
-			(at 34.29 93.98 0)
+			(at 30.48 93.98 0)
 			(effects
 				(font
@@
 			)
 		)
-		(property "Footprint" ""
+		(property "Footprint" "Fuse:Fuse_1206_3216Metric_Pad1.42x1.75mm_HandSolder"
 			(at 63.5 167.64 0)
 			(effects
@@
 			)
 		)
-		(property "Footprint" ""
+		(property "Footprint" "Capacitor_SMD:C_0805_2012Metric_Pad1.18x1.45mm_HandSolder"
 			(at 29.21 45.72 0)
 			(effects
@@
 	(symbol
 		(lib_id "power:+5V")
-		(at 34.29 83.82 0)
+		(at 30.48 83.82 0)
 		(unit 1)
 		(exclude_from_sim no)
@@
 		(fields_autoplaced yes)
 		(property "Reference" "#PWR05"
-			(at 34.29 87.63 0)
+			(at 30.48 87.63 0)
 			(effects
 				(font
@@
 		)
 		(property "Value" "+5V"
-			(at 34.29 78.74 0)
+			(at 30.48 78.74 0)
 			(effects
 				(font
@@
 		)
 		(property "Footprint" ""
-			(at 34.29 83.82 0)
+			(at 30.48 83.82 0)
 			(effects
 				(font
@@
 		)
 		(property "Datasheet" ""
-			(at 34.29 83.82 0)
+			(at 30.48 83.82 0)
 			(effects
 				(font
@@
 		)
 		(property "Description" "Power symbol creates a global label with name \"+5V\""
-			(at 34.29 83.82 0)
+			(at 30.48 83.82 0)
 			(effects
 				(font
@@
 			)
 		)
-		(property "Footprint" ""
+		(property "Footprint" "random-keyboard-parts:Reset_Pretty-Mask"
 			(at 27.94 120.65 90)
 			(effects
@@
 	)
 	(symbol
+		(lib_id "Device:C_Small")
+		(at 13.97 88.9 0)
+		(unit 1)
+		(exclude_from_sim no)
+		(in_bom yes)
+		(on_board yes)
+		(dnp no)
+		(fields_autoplaced yes)
+		(property "Reference" "C8"
+			(at 16.51 87.6362 0)
+			(effects
+				(font
+					(size 1.27 1.27)
+				)
+				(justify left)
+			)
+		)
+		(property "Value" "0.1uF"
+			(at 16.51 90.1762 0)
+			(effects
+				(font
+					(size 1.27 1.27)
+				)
+				(justify left)
+			)
+		)
+		(property "Footprint" "Capacitor_SMD:C_0805_2012Metric_Pad1.18x1.45mm_HandSolder"
+			(at 13.97 88.9 0)
+			(effects
+				(font
+					(size 1.27 1.27)
+				)
+				(hide yes)
+			)
+		)
+		(property "Datasheet" "~"
+			(at 13.97 88.9 0)
+			(effects
+				(font
+					(size 1.27 1.27)
+				)
+				(hide yes)
+			)
+		)
+		(property "Description" "Unpolarized capacitor, small symbol"
+			(at 13.97 88.9 0)
+			(effects
+				(font
+					(size 1.27 1.27)
+				)
+				(hide yes)
+			)
+		)
+		(pin "1"
+		)
+		(pin "2"
+		)
+		(instances
+			(project "PCBv1"
+				(path "/8d9d261d-9d52-405a-a0e1-e850188e3e4c"
+					(reference "C8")
+					(unit 1)
+				)
+			)
+		)
+	)
+	(symbol
 		(lib_id "Device:R_Small")
 		(at 60.96 189.23 180)
@@
 			)
 		)
-		(property "Footprint" ""
+		(property "Footprint" "Resistor_SMD:R_0805_2012Metric_Pad1.20x1.40mm_HandSolder"
 			(at 60.96 189.23 0)
 			(effects

Commit message: san
Connections:
- net at C7.2, U1.16 (XTAL2), Y1.3: no longer C6.2, U1.17 (XTAL1), Y1.1
- new net: C6.2, U1.17 (XTAL1), Y1.1
Changed lines of the file:
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@@
-	)
-	(junction
-		(at 50.8 44.45)
-		(diameter 0)
-		(color 0 0 0 0)
 	)
 	(junction
@@
 	(junction
 		(at 26.67 45.72)
-		(diameter 0)
-		(color 0 0 0 0)
-	)
-	(junction
-		(at 50.8 39.37)
 		(diameter 0)
 		(color 0 0 0 0)
@@
 	(wire
 		(pts
-			(xy 41.91 39.37) (xy 50.8 39.37)
+			(xy 41.91 39.37) (xy 53.34 39.37)
 		)
 		(stroke
@@
 	(wire
 		(pts
-			(xy 50.8 39.37) (xy 53.34 39.37)
-		)
-		(stroke
-			(width 0)
-			(type default)
-		)
-	)
-	(wire
-		(pts
 			(xy 66.04 21.59) (xy 66.04 26.67)
 		)
@@
 	(wire
 		(pts
-			(xy 50.8 44.45) (xy 53.34 44.45)
-		)
-		(stroke
-			(width 0)
-			(type default)
-		)
-	)
-	(wire
-		(pts
 			(xy 30.48 86.36) (xy 38.1 86.36)
 		)
@@
 	(wire
 		(pts
-			(xy 50.8 39.37) (xy 50.8 44.45)
-		)
-		(stroke
-			(width 0)
-			(type default)
-		)
-	)
-	(wire
-		(pts
 			(xy 68.58 26.67) (xy 71.12 26.67)
 		)
@@
 	(wire
 		(pts
-			(xy 50.8 44.45) (xy 41.91 44.45)
-		)
-		(stroke
+			(xy 41.91 44.45) (xy 53.34 44.45)
+		)
+		(stroke

Commit message: maybe done but probs not
Parts:
- removed C8: 0.1uF, Capacitor_SMD:C_0805_2012Metric_Pad1.18x1.45mm_HandSolder, symbol Device:C_Small
Connections:
- net GND: now also SW2.2; no longer SW2. (2)
- net RESET: now also SW2.1; no longer SW2. (2)
- net VCC: no longer D1.2 (I/O1), R7.1, USB1.6 (DP1), USB1.8 (DP2)
- net col6: now also U1.38 (PF5); no longer U1.36 (PF7)
- net row0: now also U1.39 (PF4); no longer U1.1 (PE6)
- net row1: now also U1.40 (PF1); no longer U1.38 (PF5)
- net row3: now also U1.1 (PE6); no longer U1.40 (PF1)
- net row4: now also U1.36 (PF7); no longer U1.39 (PF4)
- net DN: now reaches D1.3 (I/O2), R6.1, USB1.5 (DN2), USB1.7 (DN1)
- new net DP: D1.2 (I/O1), R7.1, USB1.6 (DP1), USB1.8 (DP2)
