File: matrix.kicad_sch (KiCad schematic)
At the start: 0 parts

Commit message: rah stuff
Parts:
- added D10, D11, D12, D13, D14, D15, D16, D17, D18, D19, D2, D20, D21, D22, D23, D24, D25, D26, D27, D28, D29, D3, D30, D31, D32, D33, D34, D35, D36, D37, D38, D39, D4, D40, D41, D42, D43, D44, D45, D46, D47, D48, D49, D5, D50, D51, D52, D53, D54, D55, D56, D57, D58, D59, D6, D60, D61, D62, D63, D64, D65, D66, D67, D68, D69, D7, D8, D9: D, symbol Device:D
- added SW1: SW_Push, `~, symbol Switch:SW_Push
- added SW10: SW_Push, #8, symbol Switch:SW_Push
- added SW11: SW_Push, #9, symbol Switch:SW_Push
- added SW12: SW_Push, #0, symbol Switch:SW_Push
- added SW13: SW_Push, -_, symbol Switch:SW_Push
- added SW14: SW_Push, =+, symbol Switch:SW_Push
- added SW15: SW_Push, BSPC, symbol Switch:SW_Push
- added SW16: SW_Push, PAUSE, symbol Switch:SW_Push
- added SW17: SW_Push, TAB, symbol Switch:SW_Push
- added SW18: SW_Push, Q, symbol Switch:SW_Push
- added SW19: SW_Push, W, symbol Switch:SW_Push
- added SW20: SW_Push, E, symbol Switch:SW_Push
- added SW21: SW_Push, R, symbol Switch:SW_Push
- added SW22: SW_Push, T, symbol Switch:SW_Push
- added SW23: SW_Push, Y, symbol Switch:SW_Push
- added SW24: SW_Push, U, symbol Switch:SW_Push
- added SW25: SW_Push, I, symbol Switch:SW_Push
- added SW26: SW_Push, O, symbol Switch:SW_Push
- added SW27: SW_Push, P, symbol Switch:SW_Push
- added SW28: SW_Push, [{, symbol Switch:SW_Push
- added SW29: SW_Push, ]}, symbol Switch:SW_Push
- added SW3: SW_Push, #1, symbol Switch:SW_Push
- added SW30: SW_Push, \|, symbol Switch:SW_Push
- added SW31: SW_Push, NEXT, symbol Switch:SW_Push
- added SW32: SW_Push, CPSLCK, symbol Switch:SW_Push
- added SW33: SW_Push, A, symbol Switch:SW_Push
- added SW34: SW_Push, S, symbol Switch:SW_Push
- added SW35: SW_Push, D, symbol Switch:SW_Push
- added SW36: SW_Push, F, symbol Switch:SW_Push
- added SW37: SW_Push, G, symbol Switch:SW_Push
- added SW38: SW_Push, H, symbol Switch:SW_Push
- added SW39: SW_Push, J, symbol Switch:SW_Push
- added SW4: SW_Push, #2, symbol Switch:SW_Push
- added SW40: SW_Push, K, symbol Switch:SW_Push
- added SW41: SW_Push, L, symbol Switch:SW_Push
- added SW42: SW_Push, ;:, symbol Switch:SW_Push
- added SW43: SW_Push, '", symbol Switch:SW_Push
- added SW44: SW_Push, ENTR, symbol Switch:SW_Push
- added SW45: SW_Push, PRVS, symbol Switch:SW_Push
- added SW46, SW57: SW_Push, SHFT, symbol Switch:SW_Push
- added SW47: SW_Push, Z, symbol Switch:SW_Push
- added SW48: SW_Push, X, symbol Switch:SW_Push
- added SW49: SW_Push, C, symbol Switch:SW_Push
- added SW5: SW_Push, #3, symbol Switch:SW_Push
- added SW50: SW_Push, V, symbol Switch:SW_Push
- added SW51: SW_Push, B, symbol Switch:SW_Push
- added SW52: SW_Push, N, symbol Switch:SW_Push
- added SW53: SW_Push, M, symbol Switch:SW_Push
- added SW54: SW_Push, ,<, symbol Switch:SW_Push
- added SW55: SW_Push, .>, symbol Switch:SW_Push
- added SW56: SW_Push, /?, symbol Switch:SW_Push
- added SW58: SW_Push, UP, symbol Switch:SW_Push
- added SW59: SW_Push, DEL, symbol Switch:SW_Push
- added SW6: SW_Push, #4, symbol Switch:SW_Push
- added SW60, SW66: SW_Push, CTRL, symbol Switch:SW_Push
- added SW61: SW_Push, WIN, symbol Switch:SW_Push
- added SW62, SW64: SW_Push, ALT, symbol Switch:SW_Push
- added SW63: SW_Push, SPC, symbol Switch:SW_Push
- added SW65: SW_Push, FN, symbol Switch:SW_Push
- added SW67: SW_Push, LEFT, symbol Switch:SW_Push
- added SW68: SW_Push, DOWN, symbol Switch:SW_Push
- added SW69: SW_Push, RIGHT, symbol Switch:SW_Push
- added SW7: SW_Push, #5, symbol Switch:SW_Push
- added SW8: SW_Push, #6, symbol Switch:SW_Push
- added SW9: SW_Push, #7, symbol Switch:SW_Push
Connections:
- new net: D14.2 (A), SW14.1
- new net: D17.2 (A), SW17.1
- new net: D27.2 (A), SW27.1
- new net: D38.2 (A), SW38.1
- new net: D25.2 (A), SW25.1
- new net: D4.2 (A), SW4.1
- new net: D29.2 (A), SW29.1
- new net: D50.2 (A), SW50.1
- new net: D15.2 (A), SW15.1
- new net: D8.2 (A), SW8.1
- new net: D68.2 (A), SW68.1
- new net: D60.2 (A), SW60.1
- new net: D40.2 (A), SW40.1
- new net: D22.2 (A), SW22.1
- new net: D19.2 (A), SW19.1
- new net: D34.2 (A), SW34.1
- new net: D43.2 (A), SW43.1
- new net: D49.2 (A), SW49.1
- new net: D42.2 (A), SW42.1
- new net: D21.2 (A), SW21.1
- new net: D28.2 (A), SW28.1
- new net: D65.2 (A), SW65.1
- new net: D23.2 (A), SW23.1
- new net: D12.2 (A), SW12.1
- new net: D52.2 (A), SW52.1
- new net: D9.2 (A), SW9.1
- new net: D2.2 (A), SW1.1
- new net: D5.2 (A), SW5.1
- new net: D10.2 (A), SW10.1
- new net: D55.2 (A), SW55.1
- new net: D54.2 (A), SW54.1
- new net: D45.2 (A), SW45.1
- new net: D7.2 (A), SW7.1
- new net: D37.2 (A), SW37.1
- new net: D3.2 (A), SW3.1
- new net: D64.2 (A), SW64.1
- new net: D24.2 (A), SW24.1
- new net: D63.2 (A), SW63.1
- new net: D20.2 (A), SW20.1
- new net: D58.2 (A), SW58.1
- new net: D18.2 (A), SW18.1
- new net: D48.2 (A), SW48.1
- new net: D36.2 (A), SW36.1
- new net: D59.2 (A), SW59.1
- new net: D26.2 (A), SW26.1
- new net: D56.2 (A), SW56.1
- new net: D33.2 (A), SW33.1
- new net: D39.2 (A), SW39.1
- new net: D61.2 (A), SW61.1
- new net: D32.2 (A), SW32.1
- new net: D41.2 (A), SW41.1
- new net: D13.2 (A), SW13.1
- new net: D47.2 (A), SW47.1
- new net: D16.2 (A), SW16.1
- new net: D44.2 (A), SW44.1
- new net: D35.2 (A), SW35.1
- new net: D66.2 (A), SW66.1
- new net: D69.2 (A), SW69.1
- new net: D67.2 (A), SW67.1
- new net: D31.2 (A), SW31.1
- new net: D57.2 (A), SW57.1
- new net: D46.2 (A), SW46.1
- new net: D51.2 (A), SW51.1
- new net: D6.2 (A), SW6.1
- new net: D62.2 (A), SW62.1
- new net: D53.2 (A), SW53.1
- new net: D11.2 (A), SW11.1
- new net: D30.2 (A), SW30.1
- new net Col0: SW1.2, SW17.2, SW32.2, SW46.2, SW60.2
- new net Col1: SW18.2, SW3.2, SW33.2, SW47.2, SW61.2
- new net Col10: SW12.2, SW27.2, SW42.2, SW56.2, SW65.2
- new net Col11: SW13.2, SW28.2, SW43.2, SW66.2
- new net Col12: SW14.2, SW29.2, SW57.2, SW67.2
- new net Col13: SW15.2, SW30.2, SW44.2, SW58.2, SW68.2
- new net Col14: SW16.2, SW31.2, SW45.2, SW59.2, SW69.2
- new net Col2: SW19.2, SW34.2, SW4.2, SW48.2, SW62.2
- new net Col3: SW20.2, SW35.2, SW49.2, SW5.2
- new net Col4: SW21.2, SW36.2, SW50.2, SW6.2
- new net Col5: SW22.2, SW37.2, SW51.2, SW7.2
- new net Col6: SW23.2, SW38.2, SW52.2, SW63.2, SW8.2
- new net Col7: SW24.2, SW39.2, SW53.2, SW9.2
- new net Col8: SW10.2, SW25.2, SW40.2, SW54.2
- new net Col9: SW11.2, SW26.2, SW41.2, SW55.2, SW64.2
- new net Row0: D10.1 (K), D11.1 (K), D12.1 (K), D13.1 (K), D14.1 (K), D15.1 (K), D16.1 (K), D2.1 (K), D3.1 (K), D4.1 (K), D5.1 (K), D6.1 (K), D7.1 (K), D8.1 (K), D9.1 (K)
- new net Row1: D17.1 (K), D18.1 (K), D19.1 (K), D20.1 (K), D21.1 (K), D22.1 (K), D23.1 (K), D24.1 (K), D25.1 (K), D26.1 (K), D27.1 (K), D28.1 (K), D29.1 (K), D30.1 (K), D31.1 (K)
- new net Row2: D32.1 (K), D33.1 (K), D34.1 (K), D35.1 (K), D36.1 (K), D37.1 (K), D38.1 (K), D39.1 (K), D40.1 (K), D41.1 (K), D42.1 (K), D43.1 (K), D44.1 (K), D45.1 (K)
- new net Row3: D46.1 (K), D47.1 (K), D48.1 (K), D49.1 (K), D50.1 (K), D51.1 (K), D52.1 (K), D53.1 (K), D54.1 (K), D55.1 (K), D56.1 (K), D57.1 (K), D58.1 (K), D59.1 (K)
- new net Row4: D60.1 (K), D61.1 (K), D62.1 (K), D63.1 (K), D64.1 (K), D65.1 (K), D66.1 (K), D67.1 (K), D68.1 (K), D69.1 (K)

Commit message: some progress
Parts:
- SW1: value SW_Push -> `~; footprint `~ -> (none)
- SW10: value SW_Push -> #8; footprint #8 -> (none)
- SW11: value SW_Push -> #9; footprint #9 -> (none)
- SW12: value SW_Push -> #0; footprint #0 -> (none)
- SW13: value SW_Push -> -_; footprint -_ -> (none)
- SW14: value SW_Push -> =+; footprint =+ -> (none)
- SW15: value SW_Push -> BSPC; footprint BSPC -> (none)
- SW16: value SW_Push -> PAUSE; footprint PAUSE -> (none)
- SW17: value SW_Push -> TAB; footprint TAB -> (none)
- SW18: value SW_Push -> Q; footprint Q -> (none)
- SW19: value SW_Push -> W; footprint W -> (none)
- SW20: value SW_Push -> E; footprint E -> (none)
- SW21: value SW_Push -> R; footprint R -> (none)
- SW22: value SW_Push -> T; footprint T -> (none)
- SW23: value SW_Push -> Y; footprint Y -> (none)
- SW24: value SW_Push -> U; footprint U -> (none)
- SW25: value SW_Push -> I; footprint I -> (none)
- SW26: value SW_Push -> O; footprint O -> (none)
- SW27: value SW_Push -> P; footprint P -> (none)
- SW28: value SW_Push -> [{; footprint [{ -> (none)
- SW29: value SW_Push -> ]}; footprint ]} -> (none)
- SW3: value SW_Push -> #1; footprint #1 -> (none)
- SW30: value SW_Push -> \|; footprint \| -> (none)
- SW31: value SW_Push -> NEXT; footprint NEXT -> (none)
- SW32: value SW_Push -> CPSLCK; footprint CPSLCK -> (none)
- SW33: value SW_Push -> A; footprint A -> (none)
- SW34: value SW_Push -> S; footprint S -> (none)
- SW35: value SW_Push -> D; footprint D -> (none)
- SW36: value SW_Push -> F; footprint F -> (none)
- SW37: value SW_Push -> G; footprint G -> (none)
- SW38: value SW_Push -> H; footprint H -> (none)
- SW39: value SW_Push -> J; footprint J -> (none)
- SW4: value SW_Push -> #2; footprint #2 -> (none)
- SW40: value SW_Push -> K; footprint K -> (none)
- SW41: value SW_Push -> L; footprint L -> (none)
- SW42: value SW_Push -> ;:; footprint ;: -> (none)
- SW43: value SW_Push -> '"; footprint '" -> (none)
- SW44: value SW_Push -> ENTR; footprint ENTR -> (none)
- SW45: value SW_Push -> PRVS; footprint PRVS -> (none)
- SW46, SW57: value SW_Push -> SHFT; footprint SHFT -> (none)
- SW47: value SW_Push -> Z; footprint Z -> (none)
- SW48: value SW_Push -> X; footprint X -> (none)
- SW49: value SW_Push -> C; footprint C -> (none)
- SW5: value SW_Push -> #3; footprint #3 -> (none)
- SW50: value SW_Push -> V; footprint V -> (none)
- SW51: value SW_Push -> B; footprint B -> (none)
- SW52: value SW_Push -> N; footprint N -> (none)
- SW53: value SW_Push -> M; footprint M -> (none)
- SW54: value SW_Push -> ,<; footprint ,< -> (none)
- SW55: value SW_Push -> .>; footprint .> -> (none)
- SW56: value SW_Push -> /?; footprint /? -> (none)
- SW58: value SW_Push -> UP; footprint UP -> (none)
- SW59: value SW_Push -> DEL; footprint DEL -> (none)
- SW6: value SW_Push -> #4; footprint #4 -> (none)
- SW60, SW66: value SW_Push -> CTRL; footprint CTRL -> (none)
- SW61: value SW_Push -> WIN; footprint WIN -> (none)
- SW62, SW64: value SW_Push -> ALT; footprint ALT -> (none)
- SW63: value SW_Push -> SPC; footprint SPC -> (none)
- SW65: value SW_Push -> FN; footprint FN -> (none)
- SW67: value SW_Push -> LEFT; footprint LEFT -> (none)
- SW68: value SW_Push -> DOWN; footprint DOWN -> (none)
- SW69: value SW_Push -> RIGHT; footprint RIGHT -> (none)
- SW7: value SW_Push -> #5; footprint #5 -> (none)
- SW8: value SW_Push -> #6; footprint #6 -> (none)
- SW9: value SW_Push -> #7; footprint #7 -> (none)
Connections:
- net Col0 renamed col0
- net Col1 renamed col1
- net Col10 renamed col10
- net Col11 renamed col11
- net Col12 renamed col12
- net Col13 renamed col13
- net Col14 renamed col14
- net Col2 renamed col2
- net Col3 renamed col3
- net Col4 renamed col4
- net Col5 renamed col5
- net Col6 renamed col6
- net Col7 renamed col7
- net Col8 renamed col8
- net Col9 renamed col9
- net Row0 renamed row0
- net Row1 renamed row1
- net Row2 renamed row2
- net Row3 renamed row3
- net Row4 renamed row4

Commit message: pcb start
Parts:
- D10, D11, D12, D13, D14, D15, D16, D17, D18, D19, D2, D20, D21, D22, D23, D24, D25, D26, D27, D28, D29, D3, D30, D31, D32, D33, D34, D35, D36, D37, D38, D39, D4, D40, D41, D42, D43, D44, D45, D46, D47, D48, D49, D5, D50, D51, D52, D53, D54, D55, D56, D57, D58, D59, D6, D60, D61, D62, D63, D64, D65, D66, D67, D68, D69, D7, D8, D9: footprint (none) -> Diode_SMD:D_SOD-123
- SW1, SW10, SW11, SW12, SW13, SW14, SW16, SW18, SW19, SW20, SW21, SW22, SW23, SW24, SW25, SW26, SW27, SW28, SW29, SW3, SW31, SW33, SW34, SW35, SW36, SW37, SW38, SW39, SW4, SW40, SW41, SW42, SW43, SW45, SW47, SW48, SW49, SW5, SW50, SW51, SW52, SW53, SW54, SW55, SW56, SW58, SW59, SW6, SW64, SW65, SW66, SW67, SW68, SW69, SW7, SW8, SW9: footprint (none) -> MX_Alps_Hybrid:MX-1U-NoLED
- SW15: footprint (none) -> MX_Alps_Hybrid:MX-2U-NoLED
- SW17, SW30: footprint (none) -> MX_Alps_Hybrid:MX-1.5U-NoLED
- SW32, SW57: footprint (none) -> MX_Alps_Hybrid:MX-1.75U-NoLED
- SW44, SW46: footprint (none) -> MX_Alps_Hybrid:MX-2.25U-NoLED
- SW60, SW61, SW62: footprint (none) -> MX_Alps_Hybrid:MX-1.25U-NoLED
- SW63: footprint (none) -> MX_Alps_Hybrid:MX-6.25U-NoLED

Commit message: maybe done but probs not
Parts:
- SW1, SW10, SW11, SW12, SW13, SW14, SW16, SW18, SW19, SW20, SW21, SW22, SW23, SW24, SW25, SW26, SW27, SW28, SW29, SW3, SW31, SW33, SW34, SW35, SW36, SW37, SW38, SW39, SW4, SW40, SW41, SW42, SW43, SW45, SW47, SW48, SW49, SW5, SW50, SW51, SW52, SW53, SW54, SW55, SW56, SW58, SW59, SW6, SW64, SW65, SW66, SW67, SW68, SW69, SW7, SW8, SW9: footprint MX_Alps_Hybrid:MX-1U-NoLED -> MX_Only:MXOnly-1U-NoLED
- SW15: footprint MX_Alps_Hybrid:MX-2U-NoLED -> MX_Only:MXOnly-2U-NoLED
- SW17, SW30: footprint MX_Alps_Hybrid:MX-1.5U-NoLED -> MX_Only:MXOnly-1.5U-NoLED
- SW32, SW57: footprint MX_Alps_Hybrid:MX-1.75U-NoLED -> MX_Only:MXOnly-1.75U-NoLED
- SW44, SW46: footprint MX_Alps_Hybrid:MX-2.25U-NoLED -> MX_Only:MXOnly-2.25U-NoLED
- SW60, SW61, SW62: footprint MX_Alps_Hybrid:MX-1.25U-NoLED -> MX_Only:MXOnly-1.25U-NoLED
- SW63: footprint MX_Alps_Hybrid:MX-6.25U-NoLED -> MX_Only:MXOnly-6.25U-NoLED
