File: PCBv1.kicad_pcb (KiCad board)
At the start: 2 copper layers, 157 parts, among them J1 AVR-ISP-6, SW1 `~, SW10 #8, SW11 #9, SW12 #0, SW13 -_, SW14 =+, SW15 BSPC, SW16 PAUSE, SW17 TAB, SW18 Q, SW19 W, SW2 SW_Push_Reset, SW20 E, SW21 R, SW22 T, SW23 Y, SW24 U, SW25 I, SW26 O, SW27 P, SW28 [{, SW29 ]}, SW3 #1, SW30 \|, SW31 NEXT, SW32 CPSLCK, SW33 A, SW34 S, SW35 D, SW36 F, SW37 G, SW38 H, SW39 J, SW4 #2, SW40 K, SW41 L, SW42 ;:, SW43 '", SW44 ENTR, SW45 PRVS, SW46 SHFT, SW47 Z, SW48 X, SW49 C, SW5 #3, SW50 V, SW51 B, SW52 N, SW53 M, SW54 ,<, SW55 .>, SW56 /?, SW57 SHFT, SW58 UP, SW59 DEL, SW6 #4, SW60 CTRL, SW61 WIN, SW62 ALT, SW63 SPC, SW64 ALT, SW65 FN, SW66 CTRL, SW67 LEFT, SW68 DOWN, SW69 RIGHT, SW7 #5, SW8 #6, SW9 #7, U1 ATmega32U4-A, Y1 16MHz

Commit message: san
Parts:
- moved D31 250.2 mm to (281.0, 47.6), turned to 90 degrees
- moved D16 250.0 mm to (281.0, 28.5), turned to 90 degrees
- moved D45 249.4 mm to (281.0, 66.6), turned to 90 degrees
- moved D59 249.4 mm to (281.0, 85.7), turned to 90 degrees
- moved D69 245.6 mm to (281.0, 104.8), turned to 90 degrees
- moved D58 230.6 mm to (261.9, 85.7), turned to 90 degrees
- moved D30 228.1 mm to (257.2, 47.6), turned to 90 degrees
- moved D68 226.5 mm to (261.9, 104.7), turned to 90 degrees
- moved D15 224.4 mm to (252.4, 28.5), turned to 90 degrees
- moved D44 220.6 mm to (250.0, 66.6), turned to 90 degrees
- moved D13 209.0 mm to (204.8, 28.5), turned to 90 degrees
- moved D67 207.4 mm to (242.9, 104.7), turned to 90 degrees
- moved D29 206.5 mm to (233.4, 47.6), turned to 90 degrees
- moved D57 205.6 mm to (235.7, 85.7), turned to 90 degrees
- moved D14 199.8 mm to (223.8, 28.5), turned to 90 degrees
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Connections:
- C7 pad 2: Net-(U1-XTAL1) -> Net-(U1-XTAL2)
- U1 pad 16: Net-(U1-XTAL1) -> Net-(U1-XTAL2)
- Y1 pad 3: Net-(U1-XTAL1) -> Net-(U1-XTAL2)

Commit message: maybe done but probs not
Parts:
- removed C8: 0.1uF, Capacitor_SMD:C_0805_2012Metric_Pad1.18x1.45mm_HandSolder
- SW1, SW10, SW11, SW12, SW13, SW14, SW16, SW18, SW19, SW20, SW21, SW22, SW23, SW24, SW25, SW26, SW27, SW28, SW29, SW3, SW31, SW33, SW34, SW35, SW36, SW37, SW38, SW39, SW4, SW40, SW41, SW42, SW43, SW45, SW47, SW48, SW49, SW5, SW50, SW51, SW52, SW53, SW54, SW55, SW56, SW58, SW59, SW6, SW64, SW65, SW66, SW67, SW68, SW69, SW7, SW8, SW9: footprint MX_Alps_Hybrid:MX-1U-NoLED -> MX_Only:MXOnly-1U-NoLED
- SW15: footprint MX_Alps_Hybrid:MX-2U-NoLED -> MX_Only:MXOnly-2U-NoLED
- SW17, SW30: footprint MX_Alps_Hybrid:MX-1.5U-NoLED -> MX_Only:MXOnly-1.5U-NoLED
- SW32, SW57: footprint MX_Alps_Hybrid:MX-1.75U-NoLED -> MX_Only:MXOnly-1.75U-NoLED
- SW44, SW46: footprint MX_Alps_Hybrid:MX-2.25U-NoLED -> MX_Only:MXOnly-2.25U-NoLED
- SW60, SW61, SW62: footprint MX_Alps_Hybrid:MX-1.25U-NoLED -> MX_Only:MXOnly-1.25U-NoLED
- SW63: footprint MX_Alps_Hybrid:MX-6.25U-NoLED -> MX_Only:MXOnly-6.25U-NoLED
- moved SW2 163.4 mm to (242.4, 149.1), turned to -90 degrees
- moved C2 121.1 mm to (229.5, 144.2)
- moved R5 102.3 mm to (241.6, 142.5), turned to 180 degrees
- moved J1 92.2 mm to (181.0, 150.0)
- moved R1 91.5 mm to (212.7, 157.1)
- moved SW16 91.0 mm to (363.5, 73.0)
- moved SW30 91.0 mm to (339.7, 92.1)
- moved SW31 91.0 mm to (363.5, 92.1)
- moved SW59 91.0 mm to (363.5, 130.2)
- moved SW45 91.0 mm to (363.5, 111.1)
- moved SW69 91.0 mm to (363.5, 149.2)
- moved D10 91.0 mm to (236.1, 77.7)
- moved D11 91.0 mm to (243.2, 77.7)
- moved D13 91.0 mm to (281.3, 77.7)
- moved D14 91.0 mm to (300.4, 77.7)
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Connections:
- net Net-(D1-I/O2) renamed DN
- D1 pad 2: VCC -> DP
- R7 pad 1: VCC -> DP
- SW2 pad 1: (no net) -> RESET
- SW2 pad 2: (no net) -> GND
- U1 pad 1: row0 -> row3
- U1 pad 36: col6 -> row4
- U1 pad 38: row1 -> col6
- U1 pad 39: row4 -> row0
- U1 pad 40: row3 -> row1
- USB1 pad 6: VCC -> DP
- USB1 pad 8: VCC -> DP
Routing:
- net row0: track 0.00 -> 505.7 mm, vias 0 -> 2
- net row1: track 0.00 -> 486.7 mm, vias 0 -> 4
- net row2: track 0.00 -> 466.8 mm, vias 0 -> 4
- net row3: track 0.00 -> 422.1 mm, vias 0 -> 6
- net row4: track 0.00 -> 310.6 mm
- net GND: track 0.00 -> 285.8 mm, vias 0 -> 12
- net col0: track 0.00 -> 241.2 mm, vias 0 -> 1
- net col14: track 0.00 -> 241.0 mm, vias 0 -> 1
- net col13: track 0.00 -> 231.2 mm, vias 0 -> 1
- net col1: track 0.00 -> 227.5 mm, vias 0 -> 1
- net col12: track 0.00 -> 214.0 mm, vias 0 -> 1
- net +5V: track 0.00 -> 202.8 mm, vias 0 -> 6
- net col2: track 0.00 -> 201.3 mm, vias 0 -> 1
- net col11: track 0.00 -> 190.2 mm, vias 0 -> 1
- net col10: track 0.00 -> 174.8 mm, vias 0 -> 1
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- added copper zone on F.Cu, net GND
Other:
- board outline added: 309.6 x 101.6 mm

Commit message: more done
Parts:
- moved J1 3.05 mm to (184.0, 149.8)
Routing:
- net row0: track 505.7 -> 514.2 mm
- net row3: track 422.1 -> 429.6 mm
- net row2: track 466.8 -> 474.2 mm
- net row1: track 486.7 -> 494.0 mm
- net RESET: track 91.1 -> 84.5 mm, vias 7 -> 5
- net MISO: track 61.8 -> 67.6 mm, vias 3 -> 5
- net row4: track 310.6 -> 316.0 mm
- net MOSI: track 56.7 -> 60.6 mm
- net SCK: track 64.8 -> 61.2 mm, vias 5 -> 3
- net GND: track 285.8 -> 282.5 mm
- net +5V: track 202.8 -> 201.6 mm
- net col5: track 103.0 -> 103.7 mm
- net VCC: track 25.3 -> 24.7 mm

Commit message: small fixes
Routing:
- net DP: track 86.3 -> 84.6 mm
- net DN: track 84.3 -> 82.6 mm
- net Net-(D53-A): track 6.51 -> 7.56 mm
- net Net-(D40-A): track 6.51 -> 7.52 mm
- net Net-(D55-A): track 6.51 -> 7.52 mm
- net Net-(D50-A): track 6.51 -> 7.52 mm
- net Net-(D62-A): track 6.64 -> 7.63 mm
- net Net-(D60-A): track 6.51 -> 7.50 mm
- net Net-(D32-A): track 6.51 -> 7.46 mm
- net Net-(D44-A): track 6.51 -> 7.45 mm
- net Net-(D37-A): track 6.51 -> 7.44 mm
- net Net-(D33-A): track 6.51 -> 7.44 mm
- net Net-(D45-A): track 6.51 -> 7.43 mm
- net Net-(D61-A): track 6.51 -> 7.42 mm
- net Net-(D51-A): track 6.51 -> 7.41 mm
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